File: hardware/picones.kicad_sch (KiCad schematic)
At the start: 32 parts, among them J1 NES-CART, U1 TXS0108EPW, U10 ATtiny13A-P, U11 TXS0108EPW, U12 74HC595, U13 74HC595, U14 74HC595, U15 TMUX1574PW, U16 TMUX1574PW, U17 TMUX1574PW, U18 TMUX1574PW, U19 TMUX1574PW, U2 TXS0108EPW, U20 TMUX1574PW, U21 TMUX1574PW, U22 TXS0108EPW, U23 TXS0108EPW, U24 TXS0108EPW, U25 TXS0108EPW, U26 TXS0108EPW, U27 TXS0108EPW, U28 TXS0108EPW, U3 TXS0108EPW, U4 TXS0108EPW, U5 IS62C256AL, U6 IS62C256AL, U7 74HC02, U8 74HC04, U9 TXS0108EPW

Commit message: route attempt 1
Parts:
- removed U8: 74HC04, symbol 74xx:74HC04
- added C1, C10, C11, C12, C13, C14, C15, C16, C17, C18, C19, C2, C20, C21, C22, C23, C24, C25, C26, C27, C28, C29, C3, C30, C31, C32, C33, C34, C35, C36, C4, C40, C5, C6, C7, C8, C9: .1u, Capacitor_SMD:C_0402_1005Metric, symbol Device:C_Small
- added C37, C38, C39: 10u, Capacitor_SMD:C_0402_1005Metric, symbol Device:C_Small
- added D2, D3, D4: LED, LED_SMD:LED_1206_3216Metric_Pad1.42x1.75mm_HandSolder, symbol Device:LED
- added J2: USB_C_Receptacle_USB2.0_14P, Connector_USB:USB_C_Receptacle_GCT_USB4085, symbol Connector:USB_C_Receptacle_USB2.0_14P
- added J3: Conn_01x03, Connector_PinHeader_1.27mm:PinHeader_1x03_P1.27mm_Vertical, symbol Connector_Generic:Conn_01x03
- added JP1: Mem 1 CE to GND, Connector_PinHeader_1.00mm:PinHeader_1x02_P1.00mm_Vertical, symbol Jumper:Jumper_2_Open
- added JP2: Mem 2 CE to GND, Connector_PinHeader_1.00mm:PinHeader_1x02_P1.00mm_Vertical, symbol Jumper:Jumper_2_Open
- added JP3: Disable Mem Swapping, Connector_PinHeader_1.00mm:PinHeader_1x02_P1.00mm_Vertical, symbol Jumper:Jumper_2_Open
- added JP4: VBUS to 5v, Connector_PinHeader_1.00mm:PinHeader_1x02_P1.00mm_Vertical, symbol Jumper:Jumper_2_Open
- added JP5: Connect Pico Mem CE and WE, Connector_PinHeader_1.00mm:PinHeader_1x02_P1.00mm_Vertical, symbol Jumper:Jumper_2_Open
- added R2, R3, R4, R5, R6: 5.1k, Resistor_SMD:R_0603_1608Metric_Pad0.98x0.95mm_HandSolder, symbol Device:R_US
- added SW1: Bootsel, Button_Switch_SMD:SW_Push_1P1T_NO_Vertical_Wuerth_434133025816, symbol Switch:SW_Push
- added SW2: Reset, Button_Switch_SMD:SW_Push_1P1T_NO_Vertical_Wuerth_434133025816, symbol Switch:SW_Push
- added U27: XIAO-RP2040-DIP, Module:MOUDLE14P-XIAO-DIP-SMD, symbol Seeed_Studio_XIAO_Series:XIAO-RP2040-DIP
- A1: value Pimoroni_PGA2350 -> Waveshare Core2350b; footprint Pimoroni_PGA2350:pimoroni_pga2350 -> Pimoroni_PGA2350:waveshare_core2350b
- D1: footprint (none) -> LED_SMD:LED_1206_3216Metric_Pad1.42x1.75mm_HandSolder
- R1: value R_US -> 5.1k; footprint (none) -> Resistor_SMD:R_0603_1608Metric_Pad0.98x0.95mm_HandSolder
- U1: renamed from U7; footprint (none) -> Package_DIP:DIP-14_W7.62mm
- U21: renamed from U12; footprint (none) -> Package_SO:SOIC-16W_5.3x10.2mm_P1.27mm
- U26: renamed from U13; footprint (none) -> Package_SO:SOIC-16W_5.3x10.2mm_P1.27mm
- U28: renamed from U14; footprint (none) -> Package_SO:SOIC-16W_5.3x10.2mm_P1.27mm
- renumbered U15 to U10, U18 to U11, U17 to U12, U20 to U13, U21 to U14, U19 to U15, U9 to U16, U22 to U17, U23 to U18, U24 to U19, U6 to U2, U25 to U20, U26 to U22, U27 to U23, U28 to U24, U4 to U25, U5 to U3, U2 to U4, U3 to U5, U1 to U6, U11 to U7, U10 to U8, U16 to U9
Connections:
- net +3.3V: now also U20.3 (A2), U21.16 (VCC), U25.3 (A2), U26.16 (VCC), U28.16 (VCC), C11.1, C13.1, C15.1, C2.1, C24.1, C27.1, C29.1, C32.1, C34.1, C39.1, C4.1, C6.1, C7.1, C9.1, D4.2 (A), U27.12 (3V3)
- net +5V: now also J1.57 (~{VCS}), U1.14 (VCC), C1.1, C10.1, C12.1, C14.1, C16.1, C17.1, C18.1, C19.1, C20.1, C21.1, C22.1, C23.1, C25.1, C26.1, C28.1, C3.1, C30.1, C31.1, C33.1, C35.1, C36.1, C38.1, C5.1, C8.1, D3.2 (A), JP4.2 (B)
- net CPU_D0: now also U5.12 (B8), U7.12 (B8); no longer U5.20 (B1), U7.20 (B1)
- net CPU_D1: now also U5.13 (B7), U7.13 (B7); no longer U5.18 (B2), U7.18 (B2)
- net CPU_D2: now also U5.14 (B6), U7.14 (B6); no longer U5.17 (B3), U7.17 (B3)
- net CPU_D3: now also U5.15 (B5), U7.15 (B5); no longer U5.16 (B4), U7.16 (B4)
- net CPU_D4: now also U5.16 (B4), U7.16 (B4); no longer U5.15 (B5), U7.15 (B5)
- net CPU_D5: now also U5.17 (B3), U7.17 (B3); no longer U5.14 (B6), U7.14 (B6)
- net CPU_D6: now also U5.18 (B2), U7.18 (B2); no longer U5.13 (B7), U7.13 (B7)
- net CPU_D7: now also U5.20 (B1), U7.20 (B1); no longer U5.12 (B8), U7.12 (B8)
- net CPU_R/!W: now also U1.11, U1.12
- net GND: now also U1.7 (GND), U15.4 (D1), U21.13 (~{OE}), U21.8 (GND), U26.13 (~{OE}), U26.8 (GND), U28.13 (~{OE}), U28.8 (GND), C1.2, C10.2, C11.2, C12.2, C13.2, C14.2, C15.2, C16.2, C17.2, C18.2, C19.2, C2.2, C20.2, C21.2, C22.2, C23.2, C24.2, C25.2, C26.2, C27.2, C28.2, C3.2, C30.2, C31.2, C32.2, C33.2, C34.2, C35.2, C36.2, C37.2, C38.2, C39.2, C4.2, C40.2, C5.2, C6.2, C7.2, C8.2, C9.2, J2.A1 (GND), J2.A12 (GND), J2.B1 (GND), J2.B12 (GND), J2.S1 (SHIELD), J3.1 (Pin_1), JP1.2 (B), JP2.2 (B), JP3.1 (A), R2.2, R3.2, R4.2, R5.2, R6.2, SW1.1, SW2.1, U27.13 (GND)
- net MEM_1_!CE: now also JP1.1 (A)
- net MEM_2_!CE: now also JP2.1 (A)
- net MEM_SEL_!1/2: now also U1.8, U1.9, U10.1 (SEL), U11.1 (SEL), U12.1 (SEL), U13.1 (SEL), U14.1 (SEL), U15.1 (SEL), U9.1 (SEL), JP3.2 (B)
- net MEM_SEL_!1/2_3V3: now also U17.10 (OE), U18.10 (OE), U19.10 (OE), U20.10 (OE); no longer U22.10 (OE), U23.10 (OE), U24.10 (OE), U25.10 (OE)
- net MEM_SEL_1/!2: now also U1.10; no longer U10.1 (SEL), U11.1 (SEL), U12.1 (SEL), U13.1 (SEL), U14.1 (SEL), U15.1 (SEL), U9.1 (SEL)
- net MEM_SEL_1/!2_3V3: now also A1.24 (GPIO24), U22.10 (OE), U23.10 (OE), U24.10 (OE), U25.10 (OE); no longer U17.10 (OE), U18.10 (OE), U19.10 (OE), U20.10 (OE)
- net PICO_CPU_D0_R: now also A1.30 (GPIO30), U5.9 (A8); no longer U5.1 (A1)
- net PICO_CPU_D0_W: now also U7.9 (A8); no longer U7.1 (A1)
- net PICO_CPU_D1_R: now also A1.31 (GPIO31), U5.8 (A7); no longer U5.3 (A2)
- net PICO_CPU_D1_W: now also U7.8 (A7); no longer U7.3 (A2)
- net PICO_CPU_D2_R: now also A1.32 (GPIO32), U5.7 (A6); no longer U5.4 (A3)
- net PICO_CPU_D2_W: now also U7.7 (A6); no longer U7.4 (A3)
- net PICO_CPU_D3_R: now also A1.33 (GPIO33), U5.6 (A5); no longer U5.5 (A4)
- net PICO_CPU_D3_W: now also U7.6 (A5); no longer U7.5 (A4)
- net PICO_CPU_D4_R: now also A1.34 (GPIO34), U5.5 (A4); no longer U5.6 (A5)
- net PICO_CPU_D4_W: now also U7.5 (A4); no longer U7.6 (A5)
- net PICO_CPU_D5_R: now also A1.35 (GPIO35), U5.4 (A3); no longer U5.7 (A6)
- net PICO_CPU_D5_W: now also U7.4 (A3); no longer U7.7 (A6)
- net PICO_CPU_D6_R: now also A1.36 (GPIO36), U5.3 (A2); no longer U5.8 (A7)
- net PICO_CPU_D6_W: now also U7.3 (A2); no longer U7.8 (A7)
- net PICO_CPU_D7_R: now also A1.37 (GPIO37), U5.1 (A1); no longer U5.9 (A8)
- net PICO_CPU_D7_W: now also U7.1 (A1); no longer U7.9 (A8)
- net PICO_MEM_A0: now also U21.15 (QA)
- net PICO_MEM_A1: now also U21.1 (QB)
- net PICO_MEM_A10: now also U26.2 (QC)
- net PICO_MEM_A11: now also U26.3 (QD)
- net PICO_MEM_A12: now also U26.4 (QE)
- net PICO_MEM_A13: now also U26.5 (QF)
- net PICO_MEM_A14: now also U26.6 (QG)
- net PICO_MEM_A2: now also U21.2 (QC)
- net PICO_MEM_A3: now also U21.3 (QD)
- net PICO_MEM_A4: now also U21.4 (QE)
- net PICO_MEM_A5: now also U21.5 (QF)
- net PICO_MEM_A6: now also U21.6 (QG)
- net PICO_MEM_A7: now also U21.7 (QH)
- net PICO_MEM_A8: now also U26.15 (QA)
- net PICO_MEM_A9: now also U26.1 (QB)
- net PICO_MEM_D0: now also U28.15 (QA)
- net PICO_MEM_D1: now also U28.1 (QB)
- net PICO_MEM_D2: now also U28.2 (QC)
- net PICO_MEM_D3: now also U28.3 (QD)
- net PICO_MEM_D4: now also U28.4 (QE)
- net PICO_MEM_D5: now also U28.5 (QF)
- net PICO_MEM_D6: now also U28.6 (QG)
- net PICO_MEM_D7: now also U28.7 (QH)
- net PICO_MEM_SEL_PPU_BANK: now also A1.29 (GPIO29)
- net PPU_A10: now also U12.9 (D3)
- net PPU_A11: now also U12.12 (D4)
- net PPU_A8: now also U12.4 (D1)
- net PPU_A9: now also U12.7 (D2)
- net at U1.13: now also U1.2
- net PPU_!R: now reaches U15.7 (D2)
- net PPU_!R: now also J1.21 (~{R})
- net PPU_!W: now reaches U15.9 (D3)
- net PPU_!W: now also J1.56 (~{W})
- net PICO_PPU_!CLR: now reaches U21.10 (~{SRCLR})
- net PICO_PPU_!CLR: now also A1.40 (GPIO40_ADC0), U26.10 (~{SRCLR}), U28.10 (~{SRCLR})
- net PICO_PPU_ADDR_CLK: now reaches U21.11 (SRCLK)
- net PICO_PPU_ADDR_CLK: now also A1.42 (GPIO42_ADC2), U26.11 (SRCLK)
- net PICO_PPU_LATCH: now reaches U21.12 (RCLK)
- net PICO_PPU_LATCH: now also A1.41 (GPIO41_ADC1), U26.12 (RCLK), U28.12 (RCLK)
- net PICO_PPU_ADDR_SIN: now reaches U21.14 (SER)
- net PICO_PPU_ADDR_SIN: now also A1.43 (GPIO43_ADC3)
- net at U21.9 (QH'): now also U26.14 (SER)
- net PICO_MEM_!CE: now reaches U20.1 (A1)
- net PICO_MEM_!CE: now also A1.46 (GPIO46_ADC6), U25.1 (A1), JP5.1 (A)
- net PICO_MEM_!WE: now reaches U20.4 (A3)
- net PICO_MEM_!WE: now also A1.45 (GPIO45_ADC5), U25.4 (A3), JP5.2 (B)
- net PICO_PPU_DATA_CLK: now reaches A1.38 (GPIO38)
- net PICO_PPU_DATA_CLK: now also U28.11 (SRCLK)
- net PICO_PPU_DATA_SIN: now reaches A1.39 (GPIO39)
- net PICO_PPU_DATA_SIN: now also U28.14 (SER)
- net AUDIO_UART: now reaches A1.44 (GPIO44_ADC4)
- net AUDIO_UART: now also U27.8 (GPIO1/RX)
- net at A1.48 (BOOTSEL): now also SW1.2
- net at A1.49 (SWDIO): now also J3.3 (Pin_3)
- net USB_D-: now reaches A1.50 (USB_DM)
- net USB_D-: now also J2.A7 (D-), J2.B7 (D-)
- net at A1.51 (SWCLK): now also J3.2 (Pin_2)
- net USB_D+: now reaches A1.52 (USB_DP)
- net USB_D+: now also J2.A6 (D+), J2.B6 (D+)
- net at A1.54 (RUN): now also SW2.2
- net VBUS: now reaches A1.57 (VBUS)
- net VBUS: now also C37.1, C40.1, D2.2 (A), J2.A4 (VBUS), J2.A9 (VBUS), J2.B4 (VBUS), J2.B9 (VBUS), JP4.1 (A), U27.14 (VBUS)
- new net: J2.B5 (CC2), R5.1
- new net: J2.A5 (CC1), R6.1
- new net: D4.1 (K), R4.1
- new net: D2.1 (K), R2.1
- new net: D3.1 (K), R3.1
- no-connect marks 0 -> 11
Other:
- note added: "Cartridge Memory Banks"
- note added: "NES Memory Switches"
- note added: "Other"
- note added: "Pico"
- note added: "Pico Memory Shifters"
- note added: "Pico Shift Registers"
- moved on the sheet: A1, U10, U11, U12, U13, U14, U15, U16, U17, U18, U19, U1A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
