File: hardware/picones.kicad_pcb (KiCad board)
At the start: 2 copper layers, 11 parts, among them J1 NES-CART, U1 TXS0108EPW, U10 ATtiny13A-P, U11 TXS0108EPW, U2 TXS0108EPW, U3 TXS0108EPW, U4 TXS0108EPW, U5 IS62C256AL, U6 IS62C256AL, U9 TXS0108EPW

Commit message: route attempt 1
Parts:
- added C1: .1u, Capacitor_SMD:C_0402_1005Metric, F.Cu at (118.7, 47.0)
- added C10: .1u, Capacitor_SMD:C_0402_1005Metric, F.Cu at (44.6, 80.4)
- added C11: .1u, Capacitor_SMD:C_0402_1005Metric, F.Cu at (44.6, 82.4)
- added C12: .1u, Capacitor_SMD:C_0402_1005Metric, F.Cu at (44.6, 84.3)
- added C13: .1u, Capacitor_SMD:C_0402_1005Metric, F.Cu at (44.6, 86.3)
- added C14: .1u, Capacitor_SMD:C_0402_1005Metric, F.Cu at (44.6, 88.3)
- added C15: .1u, Capacitor_SMD:C_0402_1005Metric, F.Cu at (44.6, 90.2)
- added C16: .1u, Capacitor_SMD:C_0402_1005Metric, F.Cu at (44.6, 92.2)
- added C17: .1u, Capacitor_SMD:C_0402_1005Metric, F.Cu at (44.6, 94.2)
- added C18: .1u, Capacitor_SMD:C_0402_1005Metric, F.Cu at (44.6, 96.1)
- added C19: .1u, Capacitor_SMD:C_0402_1005Metric, F.Cu at (47.5, 80.4)
- added C2: .1u, Capacitor_SMD:C_0402_1005Metric, F.Cu at (128.9, 46.4)
- added C20: .1u, Capacitor_SMD:C_0402_1005Metric, F.Cu at (47.5, 82.4)
- added C21: .1u, Capacitor_SMD:C_0402_1005Metric, F.Cu at (47.5, 84.3)
- added C22: .1u, Capacitor_SMD:C_0402_1005Metric, F.Cu at (47.5, 86.3)
- added C23: .1u, Capacitor_SMD:C_0402_1005Metric, F.Cu at (47.5, 88.3)
- added C24: .1u, Capacitor_SMD:C_0402_1005Metric, F.Cu at (47.5, 90.2)
- added C25: .1u, Capacitor_SMD:C_0402_1005Metric, F.Cu at (47.5, 92.2)
- added C26: .1u, Capacitor_SMD:C_0402_1005Metric, F.Cu at (47.5, 94.2)
- added C27: .1u, Capacitor_SMD:C_0402_1005Metric, F.Cu at (47.5, 96.1)
- added C28: .1u, Capacitor_SMD:C_0402_1005Metric, F.Cu at (50.3, 80.4)
- added C29: .1u, Capacitor_SMD:C_0402_1005Metric, F.Cu at (50.3, 82.4)
- added C3: .1u, Capacitor_SMD:C_0402_1005Metric, F.Cu at (116.8, 57.0)
- added C30: .1u, Capacitor_SMD:C_0402_1005Metric, F.Cu at (50.3, 84.3)
- added C31: .1u, Capacitor_SMD:C_0402_1005Metric, F.Cu at (50.3, 86.3)
- added C32: .1u, Capacitor_SMD:C_0402_1005Metric, F.Cu at (50.3, 88.3)
- added C33: .1u, Capacitor_SMD:C_0402_1005Metric, F.Cu at (50.3, 90.2)
- added C34: .1u, Capacitor_SMD:C_0402_1005Metric, F.Cu at (50.3, 92.2)
- added C35: .1u, Capacitor_SMD:C_0402_1005Metric, F.Cu at (50.3, 94.2)
- added C36: .1u, Capacitor_SMD:C_0402_1005Metric, F.Cu at (50.3, 96.1)
- added C37: 10u, Capacitor_SMD:C_0402_1005Metric, F.Cu at (53.2, 80.4)
- added C38: 10u, Capacitor_SMD:C_0402_1005Metric, F.Cu at (53.2, 82.4)
- added C39: 10u, Capacitor_SMD:C_0402_1005Metric, F.Cu at (53.2, 84.3)
- added C4: .1u, Capacitor_SMD:C_0402_1005Metric, F.Cu at (123.8, 54.0)
- added C40: .1u, Capacitor_SMD:C_0402_1005Metric, F.Cu at (53.2, 86.3)
- added C5: .1u, Capacitor_SMD:C_0402_1005Metric, F.Cu at (106.7, 77.5)
- added C6: .1u, Capacitor_SMD:C_0402_1005Metric, F.Cu at (41.7, 90.2)
- added C7: .1u, Capacitor_SMD:C_0402_1005Metric, F.Cu at (41.7, 92.2)
- added C8: .1u, Capacitor_SMD:C_0402_1005Metric, F.Cu at (41.7, 94.2)
- added C9: .1u, Capacitor_SMD:C_0402_1005Metric, F.Cu at (41.7, 96.1)
- added D1: LED, LED_SMD:LED_1206_3216Metric_Pad1.42x1.75mm_HandSolder, F.Cu at (88.9, 114.9)
- added D2: LED, LED_SMD:LED_1206_3216Metric_Pad1.42x1.75mm_HandSolder, F.Cu at (151.8, 41.9)
- added D3: LED, LED_SMD:LED_1206_3216Metric_Pad1.42x1.75mm_HandSolder, F.Cu at (155.6, 41.9)
- added D4: LED, LED_SMD:LED_1206_3216Metric_Pad1.42x1.75mm_HandSolder, F.Cu at (159.4, 41.9)
- added J2: USB_C_Receptacle_USB2.0_14P, Connector_USB:USB_C_Receptacle_GCT_USB4085, F.Cu at (177.8, 42.6)
- added J3: Conn_01x03, Connector_PinHeader_1.27mm:PinHeader_1x03_P1.27mm_Vertical, F.Cu at (161.3, 81.3)
- added JP1: Mem 1 CE to GND, Connector_PinHeader_1.00mm:PinHeader_1x02_P1.00mm_Vertical, F.Cu at (121.9, 89.5)
- added JP2: Mem 2 CE to GND, Connector_PinHeader_1.00mm:PinHeader_1x02_P1.00mm_Vertical, F.Cu at (124.5, 92.1)
- added JP3: Disable Mem Swapping, Connector_PinHeader_1.00mm:PinHeader_1x02_P1.00mm_Vertical, F.Cu at (133.3, 100.3)
- added JP4: VBUS to 5v, Connector_PinHeader_1.00mm:PinHeader_1x02_P1.00mm_Vertical, F.Cu at (171.2, 48.3)
- added JP5: Connect Pico Mem CE and WE, Connector_PinHeader_1.00mm:PinHeader_1x02_P1.00mm_Vertical, F.Cu at (169.5, 87.0)
- added R1: 5.1k, Resistor_SMD:R_0603_1608Metric_Pad0.98x0.95mm_HandSolder, F.Cu at (88.6, 112.4)
- added R2: 5.1k, Resistor_SMD:R_0603_1608Metric_Pad0.98x0.95mm_HandSolder, F.Cu at (148.6, 43.8)
- added R3: 5.1k, Resistor_SMD:R_0603_1608Metric_Pad0.98x0.95mm_HandSolder, F.Cu at (156.8, 50.8)
- added R4: 5.1k, Resistor_SMD:R_0603_1608Metric_Pad0.98x0.95mm_HandSolder, F.Cu at (162.8, 43.8)
- added R5: 5.1k, Resistor_SMD:R_0603_1608Metric_Pad0.98x0.95mm_HandSolder, F.Cu at (168.3, 40.6)
- added R6: 5.1k, Resistor_SMD:R_0603_1608Metric_Pad0.98x0.95mm_HandSolder, F.Cu at (177.8, 45.4)
- added SW1: Bootsel, Button_Switch_SMD:SW_Push_1P1T_NO_Vertical_Wuerth_434133025816, F.Cu at (163.4, 62.2)
- added SW2: Reset, Button_Switch_SMD:SW_Push_1P1T_NO_Vertical_Wuerth_434133025816, F.Cu at (156.4, 62.2)
- added U12: TMUX1574PW, Package_SO:TSSOP-16_4.4x5mm_P0.65mm, F.Cu at (114.9, 96.5)
- added U13: TMUX1574PW, Package_SO:TSSOP-16_4.4x5mm_P0.65mm, F.Cu at (95.9, 104.8)
- added U14: TMUX1574PW, Package_SO:TSSOP-16_4.4x5mm_P0.65mm, F.Cu at (95.9, 96.3)
- added U15: TMUX1574PW, Package_SO:TSSOP-16_4.4x5mm_P0.65mm, F.Cu at (125.4, 95.5)
- added U16: TXS0108EPW, Package_SO:TSSOP-20_4.4x6.5mm_P0.65mm, F.Cu at (127.6, 105.4)
- added U17: TXS0108EPW, Package_SO:TSSOP-20_4.4x6.5mm_P0.65mm, F.Cu at (109.2, 57.1)
- added U18: TXS0108EPW, Package_SO:TSSOP-20_4.4x6.5mm_P0.65mm, F.Cu at (123.8, 44.5)
- added U19: TXS0108EPW, Package_SO:TSSOP-20_4.4x6.5mm_P0.65mm, F.Cu at (111.1, 74.3)
- added U20: TXS0108EPW, Package_SO:TSSOP-20_4.4x6.5mm_P0.65mm, F.Cu at (94.6, 89.5)
- added U21: 74HC595, Package_SO:SOIC-16W_5.3x10.2mm_P1.27mm, F.Cu at (135.9, 43.2)
- added U22: TXS0108EPW, Package_SO:TSSOP-20_4.4x6.5mm_P0.65mm, F.Cu at (104.1, 64.8)
- added U23: TXS0108EPW, Package_SO:TSSOP-20_4.4x6.5mm_P0.65mm, F.Cu at (118.7, 52.1)
- added U24: TXS0108EPW, Package_SO:TSSOP-20_4.4x6.5mm_P0.65mm, F.Cu at (106.0, 81.9)
- added U25: TXS0108EPW, Package_SO:TSSOP-20_4.4x6.5mm_P0.65mm, F.Cu at (86.4, 86.1)
- added U26: 74HC595, Package_SO:SOIC-16W_5.3x10.2mm_P1.27mm, F.Cu at (123.2, 78.0)
- added U28: 74HC595, Package_SO:SOIC-16W_5.3x10.2mm_P1.27mm, F.Cu at (122.6, 62.2)
- added U7: TXS0108EPW, Package_SO:TSSOP-20_4.4x6.5mm_P0.65mm, F.Cu at (154.3, 125.7)
- added U8: ATtiny13A-P, Package_DIP:DIP-8_W7.62mm, F.Cu at (85.7, 118.1)
- A1: value Pimoroni_PGA2350 -> Waveshare Core2350b; footprint Pimoroni_PGA2350:pimoroni_pga2350 -> Pimoroni_PGA2350:waveshare_core2350b
- U1: value TXS0108EPW -> 74HC02; footprint Package_SO:TSSOP-20_4.4x6.5mm_P0.65mm -> Package_DIP:DIP-14_W7.62mm
- U10: value ATtiny13A-P -> TMUX1574PW; footprint Package_DIP:DIP-8_W7.62mm -> Package_SO:TSSOP-16_4.4x5mm_P0.65mm
- U11, U9: value TXS0108EPW -> TMUX1574PW; footprint Package_SO:TSSOP-20_4.4x6.5mm_P0.65mm -> Package_SO:TSSOP-16_4.4x5mm_P0.65mm
- U2, U3: value TXS0108EPW -> IS62C256AL; footprint Package_SO:TSSOP-20_4.4x6.5mm_P0.65mm -> Package_SO:SOP-28_8.4x18.16mm_P1.27mm
- U5, U6: value IS62C256AL -> TXS0108EPW; footprint Package_SO:SOP-28_8.4x18.16mm_P1.27mm -> Package_SO:TSSOP-20_4.4x6.5mm_P0.65mm
- moved U3 88.3 mm to (91.0, 69.8)
- moved U2 77.2 mm to (91.0, 49.5)
- moved U5 58.8 mm to (163.8, 120.7), turned to -90 degrees
- moved U6 55.4 mm to (173.4, 121.9), turned to -90 degrees
- moved U11 53.5 mm to (105.4, 96.5), turned to 180 degrees
- moved U10 28.7 mm to (114.9, 104.8)
- moved A1 21.6 mm to (154.3, 95.9)
- moved U4 17.0 mm to (138.1, 124.8), turned to -90 degrees
- moved U1 15.8 mm to (132.1, 127.6), turned to 180 degrees
- moved U9 13.6 mm to (105.4, 104.8)
- moved J1 4.92 mm to (131.6, 140.8)
Connections:
- A1 pad 24: unconnected-(A1-GPIO24-Pad24) -> /MEM_SEL_1/!2_3V3
- A1 pad 29: unconnected-(A1-GPIO29-Pad29) -> /PICO_MEM_SEL_PPU_BANK
- A1 pad 30: unconnected-(A1-GPIO30-Pad30) -> /PICO_CPU_D0_R
- A1 pad 31: unconnected-(A1-GPIO31-Pad31) -> /PICO_CPU_D1_R
- A1 pad 32: unconnected-(A1-GPIO32-Pad32) -> /PICO_CPU_D2_R
- A1 pad 33: unconnected-(A1-GPIO33-Pad33) -> /PICO_CPU_D3_R
- A1 pad 34: unconnected-(A1-GPIO34-Pad34) -> /PICO_CPU_D4_R
- A1 pad 35: unconnected-(A1-GPIO35-Pad35) -> /PICO_CPU_D5_R
- A1 pad 36: unconnected-(A1-GPIO36-Pad36) -> /PICO_CPU_D6_R
- A1 pad 37: unconnected-(A1-GPIO37-Pad37) -> /PICO_CPU_D7_R
- A1 pad 38: unconnected-(A1-GPIO38-Pad38) -> /PICO_PPU_DATA_CLK
- A1 pad 39: unconnected-(A1-GPIO39-Pad39) -> /PICO_PPU_DATA_SIN
- A1 pad 40: unconnected-(A1-GPIO40_ADC0-Pad40) -> /PICO_PPU_!CLR
- A1 pad 41: unconnected-(A1-GPIO41_ADC1-Pad41) -> /PICO_PPU_LATCH
- A1 pad 42: unconnected-(A1-GPIO42_ADC2-Pad42) -> /PICO_PPU_ADDR_CLK
- A1 pad 43: unconnected-(A1-GPIO43_ADC3-Pad43) -> /PICO_PPU_ADDR_SIN
- A1 pad 44: unconnected-(A1-GPIO44_ADC4-Pad44) -> /AUDIO_UART
- A1 pad 45: unconnected-(A1-GPIO45_ADC5-Pad45) -> /PICO_MEM_!WE
- A1 pad 46: unconnected-(A1-GPIO46_ADC6-Pad46) -> /PICO_MEM_!CE
- A1 pad 48: unconnected-(A1-BOOTSEL-Pad48) -> Net-(A1-BOOTSEL)
- A1 pad 49: unconnected-(A1-SWDIO-Pad49) -> Net-(A1-SWDIO)
- A1 pad 50: unconnected-(A1-USB_DM-Pad50) -> /USB_D-
- A1 pad 51: unconnected-(A1-SWCLK-Pad51) -> Net-(A1-SWCLK)
- A1 pad 52: unconnected-(A1-USB_DP-Pad52) -> /USB_D+
- A1 pad 54: unconnected-(A1-RUN-Pad54) -> Net-(A1-RUN)
- A1 pad 57: unconnected-(A1-VBUS-Pad57) -> VBUS
- J1 pad 21: unconnected-(J1-~{R}-Pad21) -> /PPU_!R
- J1 pad 56: unconnected-(J1-~{W}-Pad56) -> /PPU_!W
- J1 pad 57: unconnected-(J1-~{VCS}-Pad57) -> +5V
- U1 pad 1: /PICO_CPU_A8 -> /ROE
- U1 pad 10: +3.3V -> /MEM_SEL_1/!2
- U1 pad 11: GND -> /CPU_R/!W
- U1 pad 13: /CPU_A14 -> Net-(U1-Pad13)
- U1 pad 14: /CPU_A13 -> +5V
- U1 pad 2: +3.3V -> Net-(U1-Pad13)
- U1 pad 3: /PICO_CPU_A9 -> /CPU_ROMSEL
- U1 pad 4: /PICO_CPU_A10 -> /WIT
- U1 pad 5: /PICO_CPU_A11 -> /CPU_R/!W
- U1 pad 6: /PICO_CPU_A12 -> /CPU_ROMSEL
- U1 pad 7: /PICO_CPU_A13 -> GND
- U1 pad 8: /PICO_CPU_A14 -> /MEM_SEL_!1/2
- U1 pad 9: /PICO_CPU_R/!W -> /MEM_SEL_!1/2
- U10 pad 1: unconnected-(U10-~{RESET}/PB5-Pad1) -> /MEM_SEL_!1/2
- U10 pad 2: /CIC_CLK -> /MEM_1_A4
- U10 pad 3: Net-(D1-A) -> /MEM_2_A4
- U10 pad 4: GND -> /PPU_A4
- U10 pad 5: /CIC_DOUT -> /MEM_1_A5
- U10 pad 6: /CIC_DIN -> /MEM_2_A5
- U10 pad 7: /CIC_RST -> /PPU_A5
- U10 pad 8: +5V -> GND
- U11 pad 1: /PICO_CPU_D0_W -> /MEM_SEL_!1/2
- U11 pad 10: /WIT_3V3 -> /MEM_2_A14
- U11 pad 11: GND -> /MEM_1_A14
- U11 pad 12: /CPU_D7 -> unconnected-(U11-D4-Pad12)
- U11 pad 13: /CPU_D6 -> unconnected-(U11-S4B-Pad13)
- U11 pad 14: /CPU_D5 -> unconnected-(U11-S4A-Pad14)
- U11 pad 15: /CPU_D4 -> GND
- U11 pad 16: /CPU_D3 -> +5V
- U11 pad 2: +3.3V -> /MEM_1_A12
- U11 pad 3: /PICO_CPU_D1_W -> /MEM_2_A12
- U11 pad 4: /PICO_CPU_D2_W -> /PPU_A12
- U11 pad 5: /PICO_CPU_D3_W -> /MEM_1_A13
- U11 pad 6: /PICO_CPU_D4_W -> /MEM_2_A13
- U11 pad 7: /PICO_CPU_D5_W -> /PPU_A13
- U11 pad 8: /PICO_CPU_D6_W -> GND
- U11 pad 9: /PICO_CPU_D7_W -> /MEM_SEL_PPU_BANK
- U2 pad 1: /PICO_CPU_A0 -> /MEM_1_A14
- U2 pad 10: +3.3V -> /MEM_1_A0
- U2 pad 11: GND -> /MEM_1_D0
- U2 pad 12: /CPU_A7 -> /MEM_1_D1
- U2 pad 13: /CPU_A6 -> /MEM_1_D2
- U2 pad 14: /CPU_A5 -> GND
- U2 pad 15: /CPU_A4 -> /MEM_1_D3
- U2 pad 16: /CPU_A3 -> /MEM_1_D4
- U2 pad 17: /CPU_A2 -> /MEM_1_D5
- U2 pad 18: /CPU_A1 -> /MEM_1_D6
- U2 pad 19: +5V -> /MEM_1_D7
- U2 pad 2: +3.3V -> /MEM_1_A12
- U2 pad 20: /CPU_A0 -> /MEM_1_!CE
- U2 pad 3: /PICO_CPU_A1 -> /MEM_1_A7
- U2 pad 4: /PICO_CPU_A2 -> /MEM_1_A6
- U2 pad 5: /PICO_CPU_A3 -> /MEM_1_A5
- U2 pad 6: /PICO_CPU_A4 -> /MEM_1_A4
- U2 pad 7: /PICO_CPU_A5 -> /MEM_1_A3
- U2 pad 8: /PICO_CPU_A6 -> /MEM_1_A2
- U2 pad 9: /PICO_CPU_A7 -> /MEM_1_A1
- U3 pad 1: /PICO_CPU_D0_R -> /MEM_2_A14
- U3 pad 10: /ROE_3V3 -> /MEM_2_A0
- U3 pad 11: GND -> /MEM_2_D0
- U3 pad 12: /CPU_D7 -> /MEM_2_D1
- U3 pad 13: /CPU_D6 -> /MEM_2_D2
- U3 pad 14: /CPU_D5 -> GND
- U3 pad 15: /CPU_D4 -> /MEM_2_D3
- U3 pad 16: /CPU_D3 -> /MEM_2_D4
- U3 pad 17: /CPU_D2 -> /MEM_2_D5
- U3 pad 18: /CPU_D1 -> /MEM_2_D6
- U3 pad 19: +5V -> /MEM_2_D7
- U3 pad 2: +3.3V -> /MEM_2_A12
- U3 pad 20: /CPU_D0 -> /MEM_2_!CE
- U3 pad 3: /PICO_CPU_D1_R -> /MEM_2_A7
- U3 pad 4: /PICO_CPU_D2_R -> /MEM_2_A6
- U3 pad 5: /PICO_CPU_D3_R -> /MEM_2_A5
- U3 pad 6: /PICO_CPU_D4_R -> /MEM_2_A4
- U3 pad 7: /PICO_CPU_D5_R -> /MEM_2_A3
- U3 pad 8: /PICO_CPU_D6_R -> /MEM_2_A2
- U3 pad 9: /PICO_CPU_D7_R -> /MEM_2_A1
- U4 pad 1: unconnected-(U4-A1-Pad1) -> /PICO_CPU_A0
- U4 pad 10: unconnected-(U4-OE-Pad10) -> +3.3V
- U4 pad 11: unconnected-(U4-GND-Pad11) -> GND
- U4 pad 12: unconnected-(U4-B8-Pad12) -> /CPU_A7
- U4 pad 13: unconnected-(U4-B7-Pad13) -> /CPU_A6
- U4 pad 14: unconnected-(U4-B6-Pad14) -> /CPU_A5
- U4 pad 15: unconnected-(U4-B5-Pad15) -> /CPU_A4
- U4 pad 16: unconnected-(U4-B4-Pad16) -> /CPU_A3
- U4 pad 17: unconnected-(U4-B3-Pad17) -> /CPU_A2
- U4 pad 18: unconnected-(U4-B2-Pad18) -> /CPU_A1
- U4 pad 19: unconnected-(U4-VCCB-Pad19) -> +5V
- U4 pad 2: unconnected-(U4-VCCA-Pad2) -> +3.3V
- U4 pad 20: unconnected-(U4-B1-Pad20) -> /CPU_A0
- U4 pad 3: unconnected-(U4-A2-Pad3) -> /PICO_CPU_A1
- U4 pad 4: unconnected-(U4-A3-Pad4) -> /PICO_CPU_A2
- U4 pad 5: unconnected-(U4-A4-Pad5) -> /PICO_CPU_A3
- U4 pad 6: unconnected-(U4-A5-Pad6) -> /PICO_CPU_A4
- U4 pad 7: unconnected-(U4-A6-Pad7) -> /PICO_CPU_A5
- U4 pad 8: unconnected-(U4-A7-Pad8) -> /PICO_CPU_A6
- U4 pad 9: unconnected-(U4-A8-Pad9) -> /PICO_CPU_A7
- U5 pad 1: unconnected-(U5-A14-Pad1) -> /PICO_CPU_D7_R
- U5 pad 10: unconnected-(U5-A0-Pad10) -> /ROE_3V3
- U5 pad 11: unconnected-(U5-I/O0-Pad11) -> GND
- U5 pad 12: unconnected-(U5-I/O1-Pad12) -> /CPU_D0
- U5 pad 13: unconnected-(U5-I/O2-Pad13) -> /CPU_D1
- U5 pad 14: unconnected-(U5-GND-Pad14) -> /CPU_D2
- U5 pad 15: unconnected-(U5-I/O3-Pad15) -> /CPU_D3
- U5 pad 16: unconnected-(U5-I/O4-Pad16) -> /CPU_D4
- U5 pad 17: unconnected-(U5-I/O5-Pad17) -> /CPU_D5
- U5 pad 18: unconnected-(U5-I/O6-Pad18) -> /CPU_D6
- U5 pad 19: unconnected-(U5-I/O7-Pad19) -> +5V
- U5 pad 2: unconnected-(U5-A12-Pad2) -> +3.3V
- U5 pad 20: unconnected-(U5-~{CE}-Pad20) -> /CPU_D7
- U5 pad 3: unconnected-(U5-A7-Pad3) -> /PICO_CPU_D6_R
- U5 pad 4: unconnected-(U5-A6-Pad4) -> /PICO_CPU_D5_R
- U5 pad 5: unconnected-(U5-A5-Pad5) -> /PICO_CPU_D4_R
- U5 pad 6: unconnected-(U5-A4-Pad6) -> /PICO_CPU_D3_R
- U5 pad 7: unconnected-(U5-A3-Pad7) -> /PICO_CPU_D2_R
- U5 pad 8: unconnected-(U5-A2-Pad8) -> /PICO_CPU_D1_R
- U5 pad 9: unconnected-(U5-A1-Pad9) -> /PICO_CPU_D0_R
- U6 pad 1: unconnected-(U6-A14-Pad1) -> /PICO_CPU_A8
- U6 pad 10: unconnected-(U6-A0-Pad10) -> +3.3V
- U6 pad 11: unconnected-(U6-I/O0-Pad11) -> GND
- U6 pad 12: unconnected-(U6-I/O1-Pad12) -> /CPU_R/!W
- U6 pad 13: unconnected-(U6-I/O2-Pad13) -> /CPU_A14
- U6 pad 14: unconnected-(U6-GND-Pad14) -> /CPU_A13
- U6 pad 15: unconnected-(U6-I/O3-Pad15) -> /CPU_A12
- U6 pad 16: unconnected-(U6-I/O4-Pad16) -> /CPU_A11
- U6 pad 17: unconnected-(U6-I/O5-Pad17) -> /CPU_A10
- U6 pad 18: unconnected-(U6-I/O6-Pad18) -> /CPU_A9
- U6 pad 19: unconnected-(U6-I/O7-Pad19) -> +5V
- U6 pad 2: unconnected-(U6-A12-Pad2) -> +3.3V
- U6 pad 20: unconnected-(U6-~{CE}-Pad20) -> /CPU_A8
- U6 pad 3: unconnected-(U6-A7-Pad3) -> /PICO_CPU_A9
- U6 pad 4: unconnected-(U6-A6-Pad4) -> /PICO_CPU_A10
- U6 pad 5: unconnected-(U6-A5-Pad5) -> /PICO_CPU_A11
- U6 pad 6: unconnected-(U6-A4-Pad6) -> /PICO_CPU_A12
- U6 pad 7: unconnected-(U6-A3-Pad7) -> /PICO_CPU_A13
- U6 pad 8: unconnected-(U6-A2-Pad8) -> /PICO_CPU_A14
- U6 pad 9: unconnected-(U6-A1-Pad9) -> /PICO_CPU_R/!W
- U9 pad 1: /PICO_CPU_CLK -> /MEM_SEL_!1/2
- U9 pad 10: +3.3V -> /MEM_2_A2
- U9 pad 11: GND -> /MEM_1_A2
- U9 pad 12: /WIT -> /PPU_A3
- U9 pad 13: /ROE -> /MEM_2_A3
- U9 pad 14: unconnected-(U9-B6-Pad14) -> /MEM_1_A3
- U9 pad 15: unconnected-(U9-B5-Pad15) -> GND
- U9 pad 16: unconnected-(U9-B4-Pad16) -> +5V
- U9 pad 2: +3.3V -> /MEM_1_A0
- U9 pad 3: /PICO_CPU_IRQ -> /MEM_2_A0
- U9 pad 4: unconnected-(U9-A3-Pad4) -> /PPU_A0
- U9 pad 5: unconnected-(U9-A4-Pad5) -> /MEM_1_A1
- U9 pad 6: unconnected-(U9-A5-Pad6) -> /MEM_2_A1
- U9 pad 7: unconnected-(U9-A6-Pad7) -> /PPU_A1
- U9 pad 8: /ROE_3V3 -> GND
- U9 pad 9: /WIT_3V3 -> /PPU_A2
Routing:
- net /MEM_SEL_1/!2_3V3: track 0.00 -> 167.6 mm, vias 0 -> 9
- net /MEM_2_!WE: track 0.00 -> 148.8 mm, vias 0 -> 4
- net /MEM_1_!WE: track 0.00 -> 145.2 mm, vias 0 -> 4
- net /PICO_MEM_!WE: track 0.00 -> 144.2 mm, vias 0 -> 2
- net /MEM_1_!CE: track 0.00 -> 130.4 mm, vias 0 -> 3
- net /PICO_MEM_!CE: track 0.00 -> 129.5 mm, vias 0 -> 1
- net /MEM_1_!OE: track 0.00 -> 121.0 mm, vias 0 -> 4
- net /MEM_SEL_!1/2_3V3: track 0.00 -> 118.5 mm, vias 0 -> 7
- net GND: track 0.00 -> 118.2 mm, vias 0 -> 54
- net /MEM_2_!OE: track 0.00 -> 118.1 mm, vias 0 -> 3
- net /MEM_2_!CE: track 0.00 -> 108.5 mm, vias 0 -> 3
- net /MEM_1_A1: track 0.00 -> 105.1 mm, vias 0 -> 2
- net /MEM_SEL_!1/2: track 0.00 -> 102.3 mm, vias 0 -> 7
- net /MEM_1_A6: track 0.00 -> 101.2 mm, vias 0 -> 2
- net /MEM_1_A5: track 0.00 -> 101.1 mm, vias 0 -> 2
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- added copper zone on B.Cu, net +3.3V
- added copper zone on F.Cu, net +5V
- added copper zone on In1.Cu, net GND
- added copper zone on In4.Cu, net GND
Other:
- board outline added: 100.1 x 112 mm
- copper layers 2 -> 6
- board text added: "3V3"
- board text added: "5V"
- board text added: "VBUS"

Commit message: v1 pcb
Parts:
- removed C10, C11, C12, C14, C15, C16, C17, C18, C19, C20, C21, C22, C24, C25, C27, C28, C29, C30, C31, C32, C33, C34, C35, C36, C40, C6, C8, C9: .1u, Capacitor_SMD:C_0402_1005Metric
- removed C39: 10u, Capacitor_SMD:C_0402_1005Metric
- moved C37 120.6 mm to (166.4, 38.7), turned to 180 degrees
- moved C13 99.8 mm to (144.3, 81.9), turned to 180 degrees
- moved C7 72.4 mm to (113.0, 79.5), turned to -90 degrees
- moved C26 71.6 mm to (118.7, 100.5), turned to -90 degrees
- moved C38 61.6 mm to (97.3, 39.4)
- moved C23 58.1 mm to (99.1, 61.4), turned to 90 degrees
Routing:
- net +5V: track 90.7 -> 122.7 mm, vias 36 -> 28
- net +3.3V: track 45.4 -> 71.0 mm, vias 20 -> 22
- net GND: track 118.2 -> 139.3 mm, vias 54 -> 186
- net /MEM_1_A1: track 105.1 -> 99.6 mm
- net /MEM_2_A8: track 63.4 -> 59.1 mm
- net /MEM_2_A13: track 55.6 -> 52.0 mm
- net /MEM_1_A13: track 65.7 -> 62.8 mm
- net /MEM_2_A12: track 59.3 -> 61.9 mm
- net /MEM_1_A0: track 95.5 -> 93.3 mm
- net /MEM_2_A14: track 55.1 -> 57.2 mm
- net /MEM_1_D2: track 79.1 -> 77.0 mm
- net /MEM_1_A11: track 66.1 -> 67.9 mm
- net /PICO_CPU_A7: track 39.6 -> 37.9 mm
- net /MEM_2_A1: track 93.8 -> 92.3 mm
- net /MEM_1_A14: track 86.5 -> 87.9 mm
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